File: KiCAD/pocketSimon.sch (KiCad schematic (older format))
At the start: 30 parts, among them Q1 ztx749, Q2 2N3904, SW1 power, SW2 blue, SW3 yellow, SW4 red, SW5 green, U1 PIC10F202

Commit message: change to schematic
Parts:
- removed R1: 56, symbol R
- added P1: ICSP, symbol CONN_01X05
- added R7: 470, symbol R
- SP1: value SPEAKER -> 150 ohm
- renumbered R2 to R1, R3 to R2, R4 to R3, R5 to R4, R6 to R5, R7 to R6
Connections:
- net GND: now also P1.3 (P3)
- net Vdd: now reaches C1.1, C2.1, R2.1, R4.1, SP1.2, SW1.2, SW2.2, SW3.2, SW4.2, SW5.2, U1.2 (Vdd)
- net Vdd: now also P1.2 (P2)
- net PCLK: now reaches D2.1 (K), R3.1, U1.4 (GP1/PCLK)
- net PCLK: now also P1.5 (P5)
- net PDAT: now reaches D5.1 (K), R5.1, U1.5 (PDAT/GP0)
- net PDAT: now also P1.4 (P4)
- net at C3.1, Q2.2 (C), R11.2: now also R7.1; no longer U1.8 (GP3/~MCLR)
- net at Q1.3 (E): now also SP1.1
- new net Vpp: P1.1 (P1), R7.2, U1.8 (GP3/~MCLR)
Changed lines of the file:
@@
 LIBS:valves
 LIBS:librairie-personnelle
+LIBS:pocketSimon-cache
 EELAYER 25 0
 EELAYER END
@@
 $EndComp
 $Comp
-L R R3
+L R R2
 U 1 1 5867E571
 P 5050 2650
-F 0 "R3" V 5130 2650 50  0000 C CNN
+F 0 "R2" V 5130 2650 50  0000 C CNN
 F 1 "1K" V 5050 2650 50  0000 C CNN
 F 2 "" V 4980 2650 50  0000 C CNN
@@
 $EndComp
 $Comp
-L R R5
+L R R4
 U 1 1 5867E5E5
 P 6550 2650
-F 0 "R5" V 6630 2650 50  0000 C CNN
+F 0 "R4" V 6630 2650 50  0000 C CNN
 F 1 "1K" V 6550 2650 50  0000 C CNN
 F 2 "" V 6480 2650 50  0000 C CNN
@@
 $EndComp
 $Comp
-L R R4
+L R R3
 U 1 1 5867E648
 P 5050 4100
-F 0 "R4" V 5130 4100 50  0000 C CNN
+F 0 "R3" V 5130 4100 50  0000 C CNN
 F 1 "1K" V 5050 4100 50  0000 C CNN
 F 2 "" V 4980 4100 50  0000 C CNN
@@
 $EndComp
 $Comp
-L R R6
+L R R5
 U 1 1 5867E6BA
 P 6550 4100
-F 0 "R6" V 6630 4100 50  0000 C CNN
+F 0 "R5" V 6630 4100 50  0000 C CNN
 F 1 "1K" V 6550 4100 50  0000 C CNN
 F 2 "" V 6480 4100 50  0000 C CNN
@@
 	7200 5050 7200 5100
 Wire Wire Line
-	6350 3600 7200 3600
-Wire Wire Line
 	7200 3600 7200 4650
 $Comp
-L R R7
+L R R6
 U 1 1 5867F5D0
 P 6900 5100
-F 0 "R7" V 6980 5100 50  0000 C CNN
+F 0 "R6" V 6980 5100 50  0000 C CNN
 F 1 "3K" V 6900 5100 50  0000 C CNN
 F 2 "" V 6830 5100 50  0000 C CNN
@@
 $EndComp
 $Comp
-L R R2
+L R R1
 U 1 1 5867F951
 P 4400 5250
-F 0 "R2" V 4480 5250 50  0000 C CNN
+F 0 "R1" V 4480 5250 50  0000 C CNN
 F 1 "10K" V 4400 5250 50  0000 C CNN
 F 2 "" V 4330 5250 50  0000 C CNN
@@
 Wire Wire Line
 	3850 5450 3850 5550
-$Comp
-L R R1
-U 1 1 58680144
-P 3650 4950
-F 0 "R1" V 3730 4950 50  0000 C CNN
-F 1 "56" V 3650 4950 50  0000 C CNN
-F 2 "" V 3580 4950 50  0000 C CNN
-F 3 "" H 3650 4950 50  0000 C CNN
-	1    3650 4950
-	0    1    1    0
-$EndComp
-Wire Wire Line
-	3800 4950 3850 4950
+Wire Wire Line
+	3450 4950 3850 4950
 Wire Wire Line
 	3850 4950 3850 5050
@@
 P 3150 4850
 F 0 "SP1" H 3050 5100 50  0000 C CNN
-F 1 "SPEAKER" H 3050 4600 50  0000 C CNN
+F 1 "150 ohm" H 3050 4600 50  0000 C CNN
 F 2 "" H 3150 4850 50  0000 C CNN
 F 3 "" H 3150 4850 50  0000 C CNN
@@
 $EndComp
 Wire Wire Line
-	3500 4950 3450 4950
-Wire Wire Line
 	3450 4750 4750 4750
 Wire Wire Line
@@
 Text Notes 7100 6850 0    60   ~ 0
 PocketSimon, rev. 2\nCopyright 2016, Jacques Deschenes\nlicence: CC-BY-SA\n
+$Comp
+L R R7
+U 1 1 58690816
+P 7050 3600
+F 0 "R7" V 7130 3600 50  0000 C CNN
+F 1 "470" V 7050 3600 50  0000 C CNN
+F 2 "" V 6980 3600 50  0000 C CNN
+F 3 "" H 7050 3600 50  0000 C CNN
+	1    7050 3600
+	0    1    1    0
+$EndComp
+Wire Wire Line
+	6900 3600 6350 3600
+$Comp
+L CONN_01X05 P1
+U 1 1 586908EF
+P 8650 4800
+F 0 "P1" H 8650 5100 50  0000 C CNN
+F 1 "ICSP" V 8750 4800 50  0000 C CNN
+F 2 "" H 8650 4800 50  0000 C CNN
+F 3 "" H 8650 4800 50  0000 C CNN
+	1    8650 4800
+	1    0    0    -1
+$EndComp
+Text Label 8450 4600 2    60   ~ 0
+Vpp
+Text Label 8450 4700 2    60   ~ 0
+Vdd
+Text Label 8450 4800 2    60   ~ 0
+Vss
+Text Label 8450 4900 2    60   ~ 0
+PDAT
+Text Label 8450 5000 2    60   ~ 0
+PCLK
+Text Label 6350 3600 0    39   ~ 0
+Vpp
+Text Label 6350 3900 0    39   ~ 0
+PDAT
+Text Label 5100 3900 0    39   ~ 0
+PCLK
+Text Label 6350 3700 0    39   ~ 0
+Vss
+Text Label 5250 3700 2    39   ~ 0
+Vdd
 $EndSCHEMATC

Commit message: modification to sofware and schematic
Connections:
- net at D3.2 (A): now also R3.2
Changed lines of the file:
@@
 Text Label 5250 3700 2    39   ~ 0
 Vdd
+Wire Wire Line
+	5050 4250 5050 4300
 $EndSCHEMATC
